Commit message: fix: Update geofence coordinates and adjust GPS publisher to reflect new location

File: src/virtual_geofence/urdf/lawnmower.urdf.xacro (robot description, xacro)
@@ -395,5 +395,5 @@
       <pose>0 0 0 0 0 0</pose>
       <visualize>false</visualize>
-      <update_rate>20</update_rate>
+      <update_rate>10</update_rate>
       <ray>
         <scan>
@@ -483,10 +483,10 @@
       <pose>0 0 0 0 0 0</pose>
       <visualize>false</visualize>
-      <update_rate>30</update_rate>
+      <update_rate>20</update_rate>
       <camera>
         <horizontal_fov>1.518</horizontal_fov>
         <image>
-          <width>640</width>
-          <height>480</height>
+          <width>320</width>
+          <height>240</height>
           <format>R8G8B8</format>
         </image>
@@ -522,6 +522,6 @@
     <parent link="base_link"/>
     <child  link="nadir_camera_link"/>
-    <!-- Centred under front half of chassis, pointing straight down -->
-    <origin xyz="0.22 0 ${-base_h/2 - 0.010}" rpy="0 ${pi/2} 0"/>
+    <!-- Moved slightly back (x=0.08) and pointing DOWN (rpy="0 -pi/2 0") -->
+    <origin xyz="0.08 0 ${-base_h/2 - 0.010}" rpy="0 ${-pi/2} 0"/>
   </joint>
   <link name="nadir_camera_optical"/>
@@ -540,5 +540,5 @@
         <!-- Wider FOV for turf coverage inspection -->
         <horizontal_fov>1.222</horizontal_fov>
-        <image><width>640</width><height>480</height><format>R8G8B8</format></image>
+        <image><width>320</width><height>240</height><format>R8G8B8</format></image>
         <clip><near>0.05</near><far>1.5</far></clip>
       </camera>

Commit message: fix: Adjust camera update rates and modify nadir camera orientation for improved performance
feat: added rviz config

File: src/virtual_geofence/urdf/lawnmower.urdf.xacro (robot description, xacro)
@@ -483,5 +483,5 @@
       <pose>0 0 0 0 0 0</pose>
       <visualize>false</visualize>
-      <update_rate>20</update_rate>
+      <update_rate>10</update_rate>
       <camera>
         <horizontal_fov>1.518</horizontal_fov>
@@ -522,6 +522,6 @@
     <parent link="base_link"/>
     <child  link="nadir_camera_link"/>
-    <!-- Moved slightly back (x=0.08) and pointing DOWN (rpy="0 -pi/2 0") -->
-    <origin xyz="0.08 0 ${-base_h/2 - 0.010}" rpy="0 ${-pi/2} 0"/>
+    <!-- Angled 45 degrees forward to troubleshoot the view while keeping position -->
+    <origin xyz="0.08 0 ${-base_h/2 - 0.010}" rpy="0 ${pi*4} 0"/>
   </joint>
   <link name="nadir_camera_optical"/>
@@ -534,9 +534,9 @@
     <sensor name="nadir_cam" type="camera">
       <gz:frame_id>nadir_camera_optical</gz:frame_id>
-      <update_rate>10</update_rate>
+      <update_rate>5</update_rate>
       <visualize>false</visualize>
       <topic>/camera/nadir</topic>
       <camera>
-        <!-- Wider FOV for turf coverage inspection -->
+        <!-- Reduced resolution for better performance -->
         <horizontal_fov>1.222</horizontal_fov>
         <image><width>320</width><height>240</height><format>R8G8B8</format></image>
