File: hardware/kicad/geofence_lawnmower.kicad_sch (KiCad schematic)
At the start: 20 parts, among them J1 Raspberry Pi 5 (J8 40-pin GPI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, U1 NEO-M8N GPS, U2 HC-SR04 (Front)

Commit message: fix: Correct schematic Y-axis convention so wires actually land on pins
The sheet rendered completely broken: every symbol was mirrored about its own
origin and not one wire touched its pin (label stubs floated in empty space
beside J1). The generator placed instances and wires assuming

    screen_y = instance_y + local_y

but KiCad draws an unrotated, unmirrored instance with

    screen_y = instance_y - local_y        (placement transform [1,0,0,-1])

because embedded lib_symbols are stored Y-up while schematic space is Y-down.

This was invisible to the previous netlist self-check because the checker
reused the generator's own (wrong) transform -- generator and checker agreed
perfectly with each other and with nothing else. The convention was therefore
re-derived from real files rather than from our own assumptions: over four
upstream KiCad demos, 48 pin/wire coincidences fit the negated-Y rule, 1 fits
the naive rule (a stray endpoint on an unconnected ICL7660 pin) and 68 are
vertically symmetric parts that cannot discriminate. That check is now
committed as check_pin_convention.py.

Rather than patch coordinates by hand, the sheet is regenerated from a new
declarative generator that works entirely in screen coordinates and negates
library geometry on emit, so a pin's on-sheet position is just
instance_origin + pin.offset.

Also fixed while rebuilding:

- F1 (10A) was shorted out by a wire bridging both its terminals. The +VMOTOR
  label now sits on the far side of the fuse, so it is genuinely in series.
- Two zero-length (degenerate) wires removed.
- 16 unused J8 pins had neither a wire nor a no_connect flag; all are now
  explicitly flagged, as are the BTS7960 R_IS/L_IS current-sense outputs.
- Zone D content and the caution notes sat on top of the worksheet title
  block (x 484-592, y 386-418 mm); the zone now clears that corner.
- The battery's positive terminal is a power_out so ERC sees the +VMOTOR rail
  as driven.

The wiring itself was checked against W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
Connections:
- net +5V: now also C1.1, C2.1, C3.1, C4.1, J1.2 (5V), U1.1 (VCC), U2.1 (VCC), U_L.1 (VCC), U_R.1 (VCC); no longer C1.2, C2.2, C3.2, C4.2
- net +VMOTOR: now also U_L.9 (B+), U_R.9 (B+); no longer BT1.2 (-), F1.1
- net GND: now also BT1.2 (-), BZ1.2 (-), C1.2, C2.2, C3.2, C4.2, D1.2 (K), D2.2 (K), J1.14 (GND), J1.20 (GND), J1.25 (GND), J1.30 (GND), J1.34 (GND), J1.39 (GND), J1.6 (GND), J1.9 (GND), R4.2, U1.2 (GND), U2.2 (GND), U_L.10 (B-), U_L.2 (GND), U_R.10 (B-), U_R.2 (GND); no longer BT1.1 (+), BZ1.1 (+), C1.1, C2.1, C3.1, C4.1, D1.1 (A), D2.1 (A), R4.1
- net GPIO12_L_RPWM: now also J1.32 (GPIO12), U_L.3 (RPWM)
- net GPIO13_L_LPWM: now also J1.33 (GPIO13), U_L.4 (LPWM)
- net GPIO14_TXD: now also J1.8 (GPIO14_TXD), U1.4 (RXD)
- net GPIO15_RXD: now also J1.10 (GPIO15_RXD), U1.3 (TXD)
- net GPIO16_R_REN: now also J1.36 (GPIO16), U_R.5 (R_EN)
- net GPIO17_BUZZER: now also BZ1.1 (+), J1.11 (GPIO17); no longer BZ1.2 (-)
- net GPIO18_R_RPWM: now also J1.12 (GPIO18), U_R.3 (RPWM)
- net GPIO19_R_LPWM: now also J1.35 (GPIO19), U_R.4 (LPWM)
- net GPIO20_L_REN: now also J1.38 (GPIO20), U_L.5 (R_EN)
- net GPIO21_L_LEN: now also J1.40 (GPIO21), U_L.6 (L_EN)
- net GPIO22_LED_GRN: now also J1.15 (GPIO22), R2.1; no longer R2.2
- net GPIO23_TRIG: now also J1.16 (GPIO23), U2.3 (TRIG)
- net GPIO24_ECHO: now also J1.18 (GPIO24), R3.2, R4.1; no longer R3.1, R4.2
- net GPIO26_R_LEN: now also J1.37 (GPIO26), U_R.6 (L_EN)
- net GPIO27_LED_RED: now also J1.13 (GPIO27), R1.1; no longer R1.2
- net at U_R.11 (M+): now also M_R.1 (+)
- net at U_R.12 (M-): now also M_R.2 (-)
- net at U_L.11 (M+): now also M_L.1 (+)
- net at U_L.12 (M-): now also M_L.2 (-)
- net at U2.4 (ECHO): now also R3.1
- new net: BT1.1 (+), F1.1
- new net: D1.1 (A), R1.2
- new net: D2.1 (A), R2.2
- no-connect marks 4 -> 20
Other:
- note added: "Battery NEGATIVE ties to the common Pi GND."
- note added: "Battery POSITIVE feeds BOTH BTS7960 modules through F1."
- note added: "NEVER power the motors from the Raspberry Pi 5V rail."
- note removed: "Battery NEGATIVE ties to common Pi GND."
- note removed: "Battery POSITIVE feeds BOTH BTS7960 modules"
- note removed: "through F1. NEVER power motors from the Pi 5V rail."

Commit message: fix: Scale schematic text for A4 printing and align the zone boxes
The sheet is A2 but goes into reports on A4, i.e. a 50% linear reduction, so
1.27mm text was landing at ~0.64mm on paper -- too small to read comfortably.
Text is now 3.0mm (pin names 2.5mm, since they have to fit inside a fixed-pitch
symbol body), which prints at ~1.5mm: slightly better than a native A4 KiCad
schematic. Symbol bodies and pin pitches were scaled to match, because a symbol
is a drawing convention, not a physical dimension -- nothing is drawn to scale
and the header still mirrors the real J8 pinout.

Layout, addressing the review comments:

- The worksheet title block is a fixed 108x32mm rectangle anchored to the
  *frame's* bottom-right corner, not the page corner: x 473.5..582,
  y 375.9..408 on A2. Assuming the page corner (x 484) is why zone D sat under
  the title block. The bounds were re-measured off the rendered sheet (count
  red-dominant canvas pixels per row/column; a border is continuous, text is
  not) and the whole content column now stops at x 470.
- Every zone box now shares the same left (18) and right (470) edge, so the
  bottom boxes align with the ones above instead of overhanging.
- The sheet heading is left-aligned with the zone boxes and moved clear of the
  frame's index band.
- Title-block fields were overflowing their ~103mm text column: a 62-character
  title and an 86-character comment. Both are shortened, and the verifier now
  checks field lengths rather than leaving it to the eye.
- Reworked the layout to use the full height of the left column, since the
  title block only constrains the bottom-right corner.

verify_schematic.py gains two checks that caught real bugs during this rework:

- Diagonal wires. Adding an orthogonal-wire rule immediately flagged four
  driver-to-motor links that a layout edit had made diagonal, which meant the
  motor pins were never aligned with the driver's M+/M-.
- Title-block field length, as above.

The text-collision estim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
Parts:
- BZ1: value Active Buzzer -> Buzzer
Other:
- note added: "BOUNDARY INDICATORS"
- note added: "Battery POSITIVE feeds both BTS7960"
- note added: "DIFFERENTIAL DRIVE -- BTS7960 + DRIVE MOTORS"
- note added: "GPS RECEIVER (UART)"
- note added: "MOTOR SUPPLY -- EXTERNAL BATTERY"
- note added: "OBSTACLE SENSOR -- HC-SR04 + 3.3V LEVEL SHIFT"
- note added: "Raspberry Pi 5 hardware interconnect -- differential drive, GPS boundary enforcement, ultrasonic obstacle avoidance"
- note added: "drivers through F1 (10A)."
- note removed: "Battery POSITIVE feeds BOTH BTS7960 modules through F1."
- note removed: "DIFFERENTIAL DRIVE -- MOTOR SYSTEM (EXTERNAL BATTERY)"
- note removed: "GPS RECEIVER (UART) & BOUNDARY INDICATORS"
- note removed: "NEVER power the motors from the Raspberry Pi 5V rail."
- note removed: "OBSTACLE SENSOR -- HC-SR04 + 3.3V LEVEL-SHIFT DIVIDER"
- note removed: "Raspberry Pi 5 Hardware Interconnect -- Differential Drive, GPS Boundary Enforcement, Ultrasonic Obstacle Avoidance"
- title: GEOFENCE -- Autonomous Smart Lawn Mower -- Hardware Interconnect -> GEOFENCE -- Lawn Mower Hardware
- moved on the sheet: BT1, BZ1, C1, C2, C3, C4, D1, D2, F1, J1, M_L, M_R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

Commit message: fix: Clear the buzzer from its zone border and fill the sheet width
Two issues from review.

The buzzer overlapped the left border of its own zone box: the circle is
centred on BZ1 and has a 6.35mm radius, so at x 330.2 it reached back to
323.85 while the zone started at 326. The indicators have been spread across a
wider zone (the buzzer now sits at 384.81, well inside), which also stops that
zone looking cramped.

The right-hand side of the sheet was largely dead margin: the drawing occupied
x 18..470 of a 594mm sheet, leaving a wide empty band with only the title block
in it. Every zone row now spans the full usable width (x 18..574) and the
content is spread to use it, so the sheet reads as a filled drawing rather than
content huddled on the left.

Making the last row full width meant it had to clear the worksheet title block
(y 375.9), which caps it at 66mm tall. It now fits because:

- the ultrasonic sensor's ref/value moved below its body instead of above,
- R4's top pin is placed exactly on the divider node, so the link wire between
  them disappeared entirely (the generator's zero-length-wire assertion caught
  this the moment it stopped being a real wire),
- R4's GND label goes out to the left, since straight down would have crossed
  the bottom of the row.

Netlist is unchanged and still matches WIRING.md terminal-for-terminal.

Note on the title block: its size is not a property of the schematic. KiCad
draws it from a worksheet template, and `page_layout_descr_file` is empty in
`geofence_lawnmower.kicad_pro`, so the built-in default (fixed 108x32mm) is in
use -- which is why it did not grow with the drawing text. A custom .kicad_wks
is possible but replaces the whole page layout including the frame and index
band, and kicanvas always renders the built-in worksheet, so such a file could
not be verified with the tooling in this repo. The README records both points.
Other:
- note added: "Battery NEGATIVE ties to Pi GND."
- note added: "Battery POSITIVE -> F1 -> +VMOTOR,"
- note added: "R3/R4: 5V x 2k/(1k+2k) = 3.33V"
- note added: "which feeds both BTS7960 drivers."
- note removed: "Battery NEGATIVE ties to the common Pi GND."
- note removed: "Battery POSITIVE feeds both BTS7960"
- note removed: "R3/R4 divider: 5V x 2k/(1k+2k) = 3.33V (matches WIRING.md)"
- note removed: "drivers through F1 (10A)."
- moved on the sheet: BT1, BZ1, C1, C2, C3, C4, D1, D2, F1, J1, M_L, M_R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
